Commit message: Rename franka gripper joints to align with the HRII names

File: config/hand.xacro (robot description, xacro)
@@ -14,10 +14,10 @@
         <!--GROUP STATES: Purpose: Define a named state for a particular group, in terms of joint values. This is useful to define states like 'folded arms'-->
         <group_state name="open" group="$(arg arm_id)_hand">
-            <joint name="$(arg arm_id)_finger_joint1" value="0.035"/>
-            <joint name="$(arg arm_id)_finger_joint2" value="0.035"/>
+            <joint name="$(arg arm_id)_franka_gripper_finger_joint1" value="0.035"/>
+            <joint name="$(arg arm_id)_franka_gripper_finger_joint2" value="0.035"/>
         </group_state>
         <group_state name="close" group="$(arg arm_id)_hand">
-            <joint name="$(arg arm_id)_finger_joint1" value="0"/>
-            <joint name="$(arg arm_id)_finger_joint2" value="0"/>
+            <joint name="$(arg arm_id)_franka_gripper_finger_joint1" value="0"/>
+            <joint name="$(arg arm_id)_franka_gripper_finger_joint2" value="0"/>
         </group_state>
         <!--END EFFECTOR: Purpose: Represent information about an end effector.-->
